File: geigerteller/geiger2.sch (EAGLE design)
At the start: 56 parts, among them J1 AVR_SPI_PRG_6PTH, Q1 NFET, Q2 MMBT5088, Q4 MMBT5088, Q5 MMBT5088, U1 ATMEGA328P, U2 MAX1555, U3 LCD-16X2SILK, U4 FT232RL-BASICSSOP, U5 MC34063SMD

Commit message: Added C7, moved battery connector
Parts:
- added C7: (no value), rcl:C-EUC0805
Connections:
- net 6V: now also C7.1
- net GND: now also C7.2
Changed lines of the file:
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@@
 <part name="GND34" library="SparkFun-Aesthetics" deviceset="GND" device=""/>
 <part name="C15" library="rcl" deviceset="C-EU" device="C0603" value="10uf"/>
+<part name="C7" library="rcl" deviceset="C-EU" device="C0805"/>
+<part name="GND9" library="SparkFun-Aesthetics" deviceset="GND" device=""/>
 </parts>
 <sheets>
@@
 <instance part="GND34" gate="1" x="-149.86" y="10.16"/>
 <instance part="C15" gate="G$1" x="-30.48" y="157.48"/>
+<instance part="C7" gate="G$1" x="-165.1" y="71.12"/>
+<instance part="GND9" gate="1" x="-165.1" y="60.96"/>
 </instances>
 <busses>
@@
 <pinref part="GND23" gate="1" pin="GND"/>
 <wire x1="-210.82" y1="60.96" x2="-210.82" y2="45.72" width="0.1524" layer="91"/>
-<wire x1="-210.82" y1="66.04" x2="-210.82" y2="60.96" width="0.1524" layer="91"/>
-<junction x="-210.82" y="60.96"/>
 </segment>
 <segment>
@@
 <segment>
 <wire x1="-111.76" y1="20.32" x2="-111.76" y2="17.78" width="0.1524" layer="91"/>
+</segment>
+<segment>
+<pinref part="C7" gate="G$1" pin="2"/>
+<pinref part="GND9" gate="1" pin="GND"/>
+<wire x1="-165.1" y1="66.04" x2="-165.1" y2="63.5" width="0.1524" layer="91"/>
 </segment>
 </net>
@@
 <wire x1="-142.24" y1="76.2" x2="-160.02" y2="76.2" width="0.1524" layer="91"/>
 <pinref part="L2" gate="G$1" pin="1"/>
-<wire x1="-160.02" y1="76.2" x2="-170.18" y2="76.2" width="0.1524" layer="91"/>
+<wire x1="-160.02" y1="76.2" x2="-165.1" y2="76.2" width="0.1524" layer="91"/>
+<wire x1="-165.1" y1="76.2" x2="-170.18" y2="76.2" width="0.1524" layer="91"/>
 <wire x1="-137.16" y1="96.52" x2="-160.02" y2="96.52" width="0.1524" layer="91"/>
 <wire x1="-160.02" y1="96.52" x2="-160.02" y2="86.36" width="0.1524" layer="91"/>
@@
 <wire x1="-149.86" y1="22.86" x2="-149.86" y2="25.4" width="0.1524" layer="91"/>
 <junction x="-149.86" y="25.4"/>
-</segment>
-</net>
+<pinref part="C7" gate="G$1" pin="1"/>
+<wire x1="-165.1" y1="76.2" x2="-165.1" y2="73.66" width="0.1524" layer="91"/>
+</segment>
+</net>
